File: thin_pcb.kicad_pcb (KiCad board)
At the start: 2 copper layers, 95.2 x 95.2 mm, 226 parts, among them J01 Conn_01x02, J02 Conn_01x02, J04 Conn_01x02, J06 Conn_01x02, J07 Conn_01x02, J08 Conn_01x02, J1 USB_B_Micro, J11 Conn_01x03, J111 Conn_01x01, J115 Conn_01x01, J12 Conn_01x03, J121 Conn_01x01, J124 Conn_01x01, J125 Conn_01x01, J13 Conn_01x03, J131 Conn_01x01, J132 Conn_01x01, J133 Conn_01x01, J134 Conn_01x01, J14 Conn_01x03, J141 Conn_01x01, J142 Conn_01x01, J143 Conn_01x01, J144 Conn_01x01, J145 Conn_01x01, J15 Conn_01x03, J151 Conn_01x01, J152 Conn_01x01, J153 Conn_01x01, J154 Conn_01x01, J16 Conn_01x03, J17 Conn_01x03, J18 Conn_01x03, J2 AudioJack4_Ground, J21 Conn_01x07, J211 Conn_01x01, J214 Conn_01x01, J215 Conn_01x01, J22 Conn_01x07, J221 Conn_01x01, J224 Conn_01x01, J23 Conn_01x07, J231 Conn_01x01, J232 Conn_01x01, J233 Conn_01x01, J234 Conn_01x01, J235 Conn_01x01, J24 Conn_01x07, J241 Conn_01x01, J242 Conn_01x01, J243 Conn_01x01, J244 Conn_01x01, J25 Conn_01x07, J251 Conn_01x01, J252 Conn_01x01, J253 Conn_01x01, J254 Conn_01x01, J255 Conn_01x01, J26 Conn_01x07, J27 Conn_01x07, J28 Conn_01x07, J3 AudioJack4_Ground, J31 Conn_01x07, J32 Conn_01x07, J33 Conn_01x07, J34 Conn_01x07, J35 Conn_01x07, J36 Conn_01x07, J37 Conn_01x07, J38 Conn_01x07, J4 Conn_01x06, J41 Conn_01x04, J42 Conn_01x04, J43 Conn_01x04, J44 Conn_01x04, J45 Conn_01x04, J46 Conn_01x04, J47 Conn_01x04, J48 Conn_01x04, J5 Conn_01x06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

Commit message: breakline
Parts:
- removed the ? at (105.4, 81.9) (x2)
- removed the REF** at (70.5, 118.7)
- removed the REF** at (70.5, 80.6)
- removed the REF** at (127.6, 153.0)
- removed the REF** at (108.6, 153.0)
- removed the REF** at (70.5, 153.0)
- removed the REF** at (128.9, 78.1)
- removed the REF** at (109.9, 78.1)
- removed the REF** at (128.9, 116.2)
- removed the REF** at (109.9, 116.2)
- removed the REF** at (109.9, 135.3)
- removed the REF** at (90.8, 135.3)
- removed the REF** at (71.8, 135.3)
- removed the REF** at (52.7, 135.3)
- removed the REF** at (52.7, 116.2)
- removed the REF** at (89.5, 97.2)
- removed the REF** at (70.5, 98.4)
- removed the REF** at (127.6, 118.7)
- removed the REF** at (108.6, 118.7)
- removed the REF** at (108.6, 98.4)
- removed the REF** at (127.6, 98.4)
- removed the REF** at (127.6, 80.6)
- added ? (x2): , , F.Cu at (105.4, 81.9)
- added REF**: BreakLine_E_2, lib:BreakLine_E_2, F.Cu at (108.6, 117.5)
- added REF**: BreakLine_E_2, lib:BreakLine_E_2, F.Cu at (108.6, 97.2)
- added REF**: BreakLine_E_2, lib:BreakLine_E_2, F.Cu at (127.6, 97.2)
- added REF**: BreakLine_E_2, lib:BreakLine_E_2, F.Cu at (127.6, 79.4)
- added REF**: BreakLine_E_2, lib:BreakLine_E_2, F.Cu at (70.5, 117.5)
- added REF**: BreakLine_E_2, lib:BreakLine_E_2, F.Cu at (70.5, 79.4)
- added REF**: BreakLine_E_1, lib:BreakLine_E_1, F.Cu at (127.6, 154.3)
- added REF**: BreakLine_E_1, lib:BreakLine_E_1, F.Cu at (108.6, 154.3)
- added REF**: BreakLine_E_1, lib:BreakLine_E_1, F.Cu at (70.5, 154.3)
- added REF**: BreakLine_E_1, lib:BreakLine_E_1, F.Cu at (127.6, 78.1)
- added REF**: BreakLine_E_1, lib:BreakLine_E_1, F.Cu at (108.6, 78.1)
- added REF**: BreakLine_E_1, lib:BreakLine_E_1, F.Cu at (127.6, 116.2)
- added REF**: BreakLine_E_1, lib:BreakLine_E_1, F.Cu at (108.6, 116.2)
- added REF**: BreakLine_E_1, lib:BreakLine_E_1, F.Cu at (108.6, 135.3)
- added REF**: BreakLine_E_1, lib:BreakLine_E_1, F.Cu at (89.5, 135.3)
- added REF**: BreakLine_E_1, lib:BreakLine_E_1, F.Cu at (70.5, 135.3)
- added REF**: BreakLine_E_1, lib:BreakLine_E_1, F.Cu at (51.4, 135.3)
- added REF**: BreakLine_E_1, lib:BreakLine_E_1, F.Cu at (51.4, 116.2)
- added REF**: BreakLine_E_2, lib:BreakLine_E_2, F.Cu at (70.5, 97.2)
- added REF**: BreakLine_E_2, lib:BreakLine_E_2, F.Cu at (127.6, 117.5)
- REF**: value BreakLine_2_12.16_2 -> BreakLine_E_6; footprint lib:BreakLine_2_12.16_2 -> lib:BreakLine_E_6
- REF**: value BreakLine_2_4_4_2_2 -> BreakLine_E_2; footprint lib:BreakLine_2_4_4_2_2 -> lib:BreakLine_E_2
- REF**: value BreakLine_2_8_2_2 -> BreakLine_E_6; footprint lib:BreakLine_2_8_2_2 -> lib:BreakLine_E_6
- REF** (x3): value BreakLine_2_13.43_2 -> BreakLine_E_1; footprint lib:BreakLine_2_13.43_2 -> lib:BreakLine_E_1
- REF**: value BreakLine_2_4_5_2 -> BreakLine_E_5; footprint lib:BreakLine_2_4_5_2 -> lib:BreakLine_E_5
- REF** (x2): value BreakLine_2_4_5 -> BreakLine_E_4; footprint lib:BreakLine_2_4_5 -> lib:BreakLine_E_4
- REF**: value BreakLine_2_4_4_2_2 -> BreakLine_E_3; footprint lib:BreakLine_2_4_4_2_2 -> lib:BreakLine_E_3
- REF**: value BreakLine_2_4_4_4 -> BreakLine_E_3; footprint lib:BreakLine_2_4_4_4 -> lib:BreakLine_E_3
- moved REF** 16.5 mm to (108.6, 116.2), turned to 270 degrees
- moved REF** 1.32 mm to (108.6, 76.8)
- moved REF** 1.27 mm to (108.6, 97.2) (x2)
- moved REF** 1.27 mm to (108.6, 79.4)
- moved REF** 1.27 mm to (70.5, 116.2)
- moved REF** 1.27 mm to (127.6, 76.8)
- moved REF** 1.27 mm to (51.4, 97.2)
- moved REF** 1.27 mm to (51.4, 78.1)
- moved REF** 1.27 mm to (70.5, 76.8)
- moved REF** 1.27 mm to (70.5, 97.2)
Routing:
- net C6: track 209.8 -> 185.1 mm, vias 5 -> 3
- net F1: track 240.1 -> 233.1 mm
- net VCC: track 172.2 -> 167.4 mm
- net D5: track 244.3 -> 241.2 mm, vias 2 -> 1
- net B3: track 154.1 -> 151.0 mm, vias 2 -> 3
- net B2: track 272.6 -> 269.8 mm
- net B4: track 257.1 -> 254.5 mm
- net B1: track 176.5 -> 175.1 mm
- net D4: track 148.6 -> 147.3 mm
- net D2: track 245.9 -> 244.7 mm
- net D0: track 164.5 -> 163.5 mm
- net E6: track 147.7 -> 146.8 mm
- net Net-(D23-Pad2): track 24.4 -> 23.6 mm
- net F0: track 148.0 -> 147.2 mm
- net Net-(D13-Pad2): track 20.4 -> 21.1 mm
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Other:
- board outline removed

Commit message: gnd area
Parts:
- removed the ? at (105.4, 81.9) (x2)
- added ? (x2): , , F.Cu at (105.4, 81.9)
Routing:
- net D0: track 163.5 -> 166.9 mm
- net B4: track 254.5 -> 251.4 mm
- net D1: track 142.0 -> 144.8 mm
- net D2: track 244.7 -> 242.8 mm
- net B0: track 220.6 -> 222.4 mm
- net F4: track 194.6 -> 195.9 mm
- net B6: track 295.2 -> 296.5 mm
- net F6: track 136.3 -> 137.3 mm
- net F5: track 133.7 -> 134.5 mm
- net D3: track 148.6 -> 149.4 mm
- net C7: track 105.0 -> 105.6 mm
- net B7: track 171.7 -> 172.3 mm
- net D7: track 138.3 -> 137.8 mm
- net GND: vias 11 -> 128
- net (no net): vias 0 -> 1
- added copper zone on B.Cu, net GND
- added copper zone on F.Cu, net GND
Other:
- board outline added: 95.2 x 95.2 mm
